File: hellen121vag.kicad_pcb (KiCad board)
At the start: 4 copper layers, 164 x 118 mm, 125 parts, among them J1 USB_B_Mini, J10 AudioJack_THR, J2 Conn_01x01, J3 Conn_01x01, J4 Conn_01x01, J5 Conn_01x01, J6 Conn_01x01, J7 Conn_01x08, J8 Conn_01x06, M1 Module-can-0.1, M10 Module-can-0.1, M11 Module-vr-discrete-0.1, M2 Module-power5-0.2, M3 Module-mcu-0.7, M4 Module-input-0.1, M5 Module-knock-0.1, M6 Module-output-0.3, M7 Module-ign8-0.2, M8 Module-power12-0.2, M9 Module-wbo-0.3, P1 368255-2, P10 Pad, P11 Pad, P12 Pad, P13 Pad, P14 Pad, P15 Pad, P16 Pad, P17 Pad, P2 Pad, P20 Pad, P28 Pad, P3 Pad, P4 Pad, P40 Pad, P41 Pad, P43 Pad, P44 Pad, P45 Pad, P46 Pad, P48 Pad, P49 Pad, P5 Pad, P56 Pad, P6 Pad, P61 Pad, P63 Pad, P64 Pad, P66 Pad, P67 Pad, P68 Pad, P69 Pad, P7 Pad, P74 Pad, P8 Pad, P80 Pad, P9 Pad, U1 L6205PD, U2 LPS25HB, U3 MCP6002-xSN

Commit message: modifique la pcb
Parts:
- removed C1, C15, C16, C2, C6: 100n, hellen-one-common:C0603
- removed C11, C12, C13, C14, C7, C8, C9: 10u, Capacitor_SMD:C_0805_2012Metric
- removed C17: 10u, hellen-one-common:C0603
- removed D1, D3, D5, D9: 1N4148WS, hellen-one-common:SOD-323
- removed D10, D11, D12, D13, D14: B5819W, Diode_SMD:D_SOD-123
- removed D4, D6, D7, D8: LED-GREEN-0805, hellen-one-common:LED-0805
- removed F1, F2: Fuse-Pad-Pad, hellen-one-common:PAD-1206-PAD
- removed G***: LOGO, hellen-one-common:LOGO
- removed G4: DISCLAIMER, rusefi_lib:Off_Road_Disclaimer
- removed J1: USB_B_Mini, hellen-one-common:USB-MINI-B-VERTICAL
- removed J10: AudioJack_THR, hellen-one-common:Jack_3.5mm_PJ-3250-5A
- removed J2, J3, J4, J5, J6: Conn_01x01, TestPoint:TestPoint_Pad_D2.0mm
- removed J7: Conn_01x08, Connector_PinHeader_2.54mm:PinHeader_1x08_P2.54mm_Vertical
- removed J8: Conn_01x06, Connector_PinHeader_2.54mm:PinHeader_1x06_P2.54mm_Vertical
- removed M1, M10: Module-can-0.1, hellen-one-can-0.1:can
- removed M2: Module-power5-0.2, hellen-one-power5-0.2:power5
- removed M5: Module-knock-0.1, hellen-one-knock-0.1:knock
- removed M9: Module-wbo-0.3, hellen-one-wbo-0.3:wbo
- removed P10, P11, P12, P13, P14, P15, P16, P17, P2, P20, P28, P3, P4, P40, P41, P43, P44, P45, P46, P48, P49, P5, P56, P6, P61, P63, P64, P66, P67, P68, P69, P7, P74, P8, P80, P9: Pad, hellen-one-common:PAD-TH
- removed R10, R11, R12, R13, R2, R3, R4, R8, R9: Jumper-Pad-Pad, hellen-one-common:PAD-0805-PAD
- removed R16, R17: 5.1k, hellen-one-common:R0603
- removed R18, R19: 4.7k, hellen-one-common:R0603
- removed R20: 1.6k, hellen-one-common:R0603
- removed R21: 750, hellen-one-common:R0603
- removed R23: 0, hellen-one-common:R0603
- removed R6, R7: 2.7k, hellen-one-common:R0603
- removed S1, S2: Button_SPST, hellen-one-common:SMD-2_2.9x3.9x1.7
- removed U2: LPS25HB, Package_LGA:ST_HLGA-10_2.5x2.5mm_P0.6mm_LayoutBorder3x2y
- removed U3: MCP6002-xSN, Package_SO:SOIC-8_3.9x4.9mm_P1.27mm
Routing:
- net +12V_RAW: track 567.8 -> 166.6 mm, vias 18 -> 10
- net +5V: track 359.2 -> 39.4 mm, vias 4 -> 0
- net +3V3: track 198.6 -> 11.0 mm, vias 4 -> 0
- net /IN_VIGN: track 171.1 -> 0.00 mm, vias 1 -> 0
- net /VBAT: track 111.2 -> 0.00 mm, vias 4 -> 0
- net /CAN+: track 120.8 -> 25.8 mm, vias 2 -> 0
- net Net-(C17-Pad2): track 92.0 -> 0.00 mm
- net /CAN-: track 117.7 -> 26.4 mm, vias 2 -> 0
- net +12V: track 95.3 -> 5.08 mm
- net GND: track 109.8 -> 23.2 mm, vias 125 -> 49
- net /THRESHOLD_VR: track 77.2 -> 0.00 mm, vias 2 -> 0
- net /OUT_MAIN_RELAY: track 69.3 -> 0.00 mm
- net /-ETB: track 115.5 -> 47.8 mm, vias 3 -> 2
- net /+ETB: track 116.7 -> 50.3 mm, vias 3 -> 2
- net /ETB_EN: track 85.7 -> 20.6 mm, vias 1 -> 0
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- removed copper zone on B.Cu, net /OUT_INJ2
- removed copper zone on B.Cu, net Net-(J1-Pad5)
- removed copper zone on F.Cu, net Net-(J1-Pad5)
Other:
- board text removed: "+12"
- board text removed: "+3.3"
- board text removed: "+5"
- board text removed: "12V SRC"
- board text removed: "3.3"
- board text removed: "<- Knock audio"
- board text removed: "Always looking for C/C++/PHP/Java developers https://rusefi.com/s/mission"
- board text removed: "Baro"
- board text removed: "CLK"
- board text removed: "DIO"
- board text removed: "G"
- board text removed: "Hellen121vag"
- board text removed: "PROG"
- board text removed: "RESET"
- board text removed: "RST"
- board text removed: "SWD WBO"
- board text removed: "Vign"
- board text removed: "rev. d"
- board text removed: "© andreika, 2021"

Commit message: modifique la pcb
Parts:
- removed G1, G2, G3, G5: PROTO_AREA, hellen-one-common:PROTO_AREA
Routing:
- net +5V: track 39.4 -> 14.8 mm
- net Net-(G5-Pad14): track 5.08 -> 0.00 mm
- net Net-(G5-Pad13): track 5.08 -> 0.00 mm
- net Net-(G5-Pad12): track 5.08 -> 0.00 mm
- net Net-(G5-Pad10): track 5.08 -> 0.00 mm
- net Net-(G5-Pad1): track 5.08 -> 0.00 mm
- net Net-(G2-Pad14): track 5.08 -> 0.00 mm
- net Net-(G2-Pad13): track 5.08 -> 0.00 mm
- net Net-(G2-Pad12): track 5.08 -> 0.00 mm
- net Net-(G2-Pad10): track 5.08 -> 0.00 mm
- net Net-(G2-Pad1): track 5.08 -> 0.00 mm
- net Net-(G1-Pad10): track 5.08 -> 0.00 mm
- net +12V: track 5.08 -> 0.00 mm
- net GND: vias 49 -> 48
Other:
- board text removed: "GND"

Commit message: modifique la pcb
Parts:
- removed BT1: BATTERY_CR2032, Battery:BatteryHolder_Keystone_1060_1x2032
- removed C10: 10u, Capacitor_SMD:C_0805_2012Metric
- removed C3: 220n, hellen-one-common:C0603
- removed C4: 10n, hellen-one-common:C0603
- removed C5: 5.6n, hellen-one-common:C0603
- removed D2: 1N4148WS, hellen-one-common:SOD-323
- removed G6: LOGO, hellen-one-common:LOGO
- removed M11: Module-vr-discrete-0.1, hellen-one-vr-discrete-0.1:vr-discrete
- removed R1: 100, hellen-one-common:R0603
- removed R22: 10k, hellen-one-common:R0603
- removed R5: 100k, hellen-one-common:R0603
- removed U1: L6205PD, hellen-one-common:SO20POWER
Routing:
- net /OUT_IGN1: track 172.0 -> 0.00 mm, vias 1 -> 0
- net /OUT_IGN3: track 169.6 -> 0.00 mm, vias 1 -> 0
- net +12V_RAW: track 166.6 -> 0.00 mm, vias 10 -> 0
- net /OUT_IGN4: track 163.7 -> 0.00 mm, vias 1 -> 0
- net /OUT_IGN2: track 146.8 -> 0.00 mm, vias 1 -> 0
- net Net-(F1-Pad1): track 140.3 -> 0.00 mm
- net /OUT_FUEL_CONSUM: track 117.7 -> 0.00 mm, vias 2 -> 0
- net /OUT_VVT2_B1: track 117.6 -> 0.00 mm
- net /OUT_IGN5: track 112.4 -> 0.00 mm
- net /OUT_IGN6: track 110.9 -> 0.00 mm, vias 1 -> 0
- net GNDA: track 104.1 -> 0.00 mm, vias 1 -> 0
- net /OUT_IGN8: track 101.1 -> 0.00 mm
- net /IN_CAM2: track 77.2 -> 0.00 mm
- net Net-(P1-Pad51): track 76.2 -> 0.00 mm, vias 1 -> 0
- net Net-(P1-Pad70): track 76.0 -> 0.00 mm, vias 1 -> 0
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Other:
- board size 164 x 118 mm -> 164 x 105.4 mm
- board text removed: "1"
- board text removed: "10"
- board text removed: "100"
- board text removed: "101"
- board text removed: "102"
- board text removed: "103"
- board text removed: "104"
- board text removed: "105"
- board text removed: "106"
- board text removed: "11"
- board text removed: "112"
- board text removed: "113"
- board text removed: "114"
- board text removed: "115"
- board text removed: "116"
- board text removed: "117"
- board text removed: "118"
- board text removed: "119"
- board text removed: "12"
- board text removed: "120"
- board text removed: "121"
- board text removed: "13"
- board text removed: "14"
- board text removed: "15"
- board text removed: "16"
- board text removed: "17"
- board text removed: "18"
- board text removed: "19"
- board text removed: "2"
- board text removed: "20"
- board text removed: "21"
- board text removed: "22"
- board text removed: "23"
- board text removed: "24"
- board text removed: "25"
- board text removed: "26"
- board text removed: "27"
- board text removed: "28"
- board text removed: "29"
- board text removed: "3"
- board text removed: "30"
- board text removed: "31"
- board text removed: "32"
- board text removed: "33"
- board text removed: "34"
- board text removed: "35"
- board text removed: "36"
- board text removed: "37"
- board text removed: "38"
- board text removed: "39"
- board text removed: "4"
- board text removed: "40"
- board text removed: "41"
- board text removed: "42"
- board text removed: "43"
- board text removed: "44"
- board text removed: "45"
- board text removed: "46"
- board text removed: "47"
- board text removed: "48"
- board text removed: "49"
- board text removed: "5"
- board text removed: "50"
- board text removed: "51"
- board text removed: "52"
- board text removed: "53"
- board text removed: "54"
- board text removed: "55"
- board text removed: "56"
- board text removed: "57"
- board text removed: "58"
- board text removed: "59"
- board text removed: "6"
- board text removed: "60"
- board text removed: "61"
- board text removed: "62"
- board text removed: "63"
- board text removed: "64"
- board text removed: "65"
- board text removed: "66"
- board text removed: "67"
- board text removed: "68"
- board text removed: "69"
- board text removed: "7"
- board text removed: "70"
- board text removed: "71"
- board text removed: "72"
- board text removed: "73"
- board text removed: "74"
- board text removed: "75"
- board text removed: "76"
- board text removed: "77"
- board text removed: "78"
- board text removed: "79"
- board text removed: "8"
- board text removed: "80"
- board text removed: "81"
- board text removed: "82"
- board text removed: "83"
- board text removed: "84"
- board text removed: "85"
- board text removed: "86"
- board text removed: "87"
- board text removed: "88"
- board text removed: "89"
- board text removed: "9"
- board text removed: "90"
- board text removed: "91"
- board text removed: "92"
- board text removed: "93"
- board text removed: "94"
- board text removed: "95"
- board text removed: "96"
- board text removed: "97"
- board text removed: "98"
- board text removed: "99"
